File: untitled.brd (EAGLE design)
At the start: 160 x 100 mm, 33 parts, among them Q1 S8050, Q2 S8050, T1 BTA26-H

Commit message: working
Parts:
- removed R11, R13: 12k, resistor:M0805
- removed S2: 5501-1LED, switch:5501-1LED
- added C9: (no value), capacitor-wima:C15B6
- added OK2: MOC3031S, optocoupler:DIL6-SMD
- added R15, R17: 220R, resistor:M0805
- added R16: 100R, resistor:M0805
- added T2: BTA26-H, triac:TOP3L-1
- C8: value 470pF -> (none); device rcl:C0805K -> capacitor-wima:C15B6
- moved C8 87.9 mm to (-58.4, -268.0)
Connections:
- new net A1_LIVE_OUT: T1.A2, T2.A2
- new net A2_LIVE_IN: R15.1, R17.1, T1.A1, T2.A1
- new net LIVE_IN: C8.1
- new net N$13: OK1.6, R15.2
- new net N$14: OK1.4, T1.G
- new net N$15: OK2.1, R16.1
- new net N$16: OK2.6, R17.2
- new net N$17: OK2.4, T2.G
- net BUTT_L: now also R12.1
- net GND: now also OK2.2
- net SW_R: now also R16.2
Changed lines of the file:
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@@
 <element name="C6" library="rcl" library_urn="urn:adsk.eagle:library:334" package="C0805" package3d_urn="urn:adsk.eagle:package:23617/2" value="10uF" x="-40.64" y="-96.52"/>
 <element name="S1" library="switch" library_urn="urn:adsk.eagle:library:380" package="5501-1LED" package3d_urn="urn:adsk.eagle:package:27757/1" value="5501-1LED" x="-30.48" y="-111.76"/>
-<element name="S2" library="switch" library_urn="urn:adsk.eagle:library:380" package="5501-1LED" package3d_urn="urn:adsk.eagle:package:27757/1" value="5501-1LED" x="-30.48" y="-134.62"/>
 <element name="R10" library="resistor" library_urn="urn:adsk.eagle:library:348" package="M0805" package3d_urn="urn:adsk.eagle:package:26079/1" value="12k" x="-40.64" y="-149.86"/>
-<element name="R11" library="resistor" library_urn="urn:adsk.eagle:library:348" package="M0805" package3d_urn="urn:adsk.eagle:package:26079/1" value="12k" x="-40.64" y="-156.21"/>
 <element name="R12" library="resistor" library_urn="urn:adsk.eagle:library:348" package="M0805" package3d_urn="urn:adsk.eagle:package:26079/1" value="12k" x="-40.64" y="-162.56"/>
-<element name="R13" library="resistor" library_urn="urn:adsk.eagle:library:348" package="M0805" package3d_urn="urn:adsk.eagle:package:26079/1" value="12k" x="-40.64" y="-168.91"/>
 <element name="C7" library="rcl" library_urn="urn:adsk.eagle:library:334" package="C0805K" package3d_urn="urn:adsk.eagle:package:23681/2" value="470pF" x="-41.91" y="-175.26"/>
-<element name="C8" library="rcl" library_urn="urn:adsk.eagle:library:334" package="C0805K" package3d_urn="urn:adsk.eagle:package:23681/2" value="470pF" x="-41.91" y="-181.61"/>
 <element name="OK1" library="optocoupler" library_urn="urn:adsk.eagle:library:320" package="DIL6-SMD" package3d_urn="urn:adsk.eagle:package:21970/1" value="MOC3031S" x="-36.83" y="-190.5">
 <attribute name="MF" value="FAIRCHILD SEMICONDUCTOR" x="-36.83" y="-190.5" size="1.778" layer="27" display="off"/>
@@
 <element name="R14" library="resistor" library_urn="urn:adsk.eagle:library:348" package="M0805" package3d_urn="urn:adsk.eagle:package:26079/1" value="100R" x="-40.64" y="-199.39"/>
 <element name="T1" library="triac" library_urn="urn:adsk.eagle:library:403" package="TOP3L-1" package3d_urn="urn:adsk.eagle:package:30152/1" value="BTA26-H" x="-60.96" y="-184.15"/>
+<element name="R15" library="resistor" library_urn="urn:adsk.eagle:library:348" package="M0805" package3d_urn="urn:adsk.eagle:package:26079/1" value="220R" x="-74.93" y="-205.74"/>
+<element name="OK2" library="optocoupler" library_urn="urn:adsk.eagle:library:320" package="DIL6-SMD" package3d_urn="urn:adsk.eagle:package:21970/1" value="MOC3031S" x="-69.85" y="-251.46">
+<attribute name="MF" value="FAIRCHILD SEMICONDUCTOR" x="-69.85" y="-214.63" size="1.778" layer="27" display="off"/>
+<attribute name="MPN" value="MOC3031SM" x="-69.85" y="-214.63" size="1.778" layer="27" display="off"/>
+<attribute name="OC_FARNELL" value="unknown" x="-69.85" y="-214.63" size="1.778" layer="27" display="off"/>
+<attribute name="OC_NEWARK" value="34C1335" x="-69.85" y="-214.63" size="1.778" layer="27" display="off"/>
+</element>
+<element name="R16" library="resistor" library_urn="urn:adsk.eagle:library:348" package="M0805" package3d_urn="urn:adsk.eagle:package:26079/1" value="100R" x="-62.23" y="-248.92"/>
+<element name="T2" library="triac" library_urn="urn:adsk.eagle:library:403" package="TOP3L-1" package3d_urn="urn:adsk.eagle:package:30152/1" value="BTA26-H" x="-60.96" y="-227.33"/>
+<element name="R17" library="resistor" library_urn="urn:adsk.eagle:library:348" package="M0805" package3d_urn="urn:adsk.eagle:package:26079/1" value="220R" x="-55.88" y="-248.92"/>
+<element name="C8" library="capacitor-wima" library_urn="urn:adsk.eagle:library:116" package="C15B6" package3d_urn="urn:adsk.eagle:package:5403/1" value="" x="-58.42" y="-267.97"/>
+<element name="C9" library="capacitor-wima" library_urn="urn:adsk.eagle:library:116" package="C15B6" package3d_urn="urn:adsk.eagle:package:5403/1" value="" x="-58.42" y="-289.56"/>
 </elements>
 <signals>
@@
 <contactref element="S1" pad="-"/>
 <contactref element="OK1" pad="2"/>
+<contactref element="OK2" pad="2"/>
 <wire x1="-40.91" y1="-175.26" x2="-36.83" y2="-195.145" width="0" layer="19" extent="1-1"/>
 <wire x1="-39.69" y1="-162.56" x2="-40.91" y2="-175.26" width="0" layer="19" extent="1-1"/>
@@
 <wire x1="-34.61" y1="57.15" x2="-40.91" y2="55.88" width="0" layer="19" extent="1-1"/>
 <wire x1="-15.51" y1="63.5" x2="-34.61" y2="57.15" width="0" layer="19" extent="1-1"/>
+<wire x1="-69.85" y1="-256.105" x2="-36.83" y2="-195.145" width="0" layer="19" extent="1-1"/>
 </signal>
 <signal name="+3V3">
@@
 <contactref element="S1" pad="1A"/>
 <contactref element="S1" pad="1B"/>
-<wire x1="-30.48" y1="-115.57" x2="-42.91" y2="-175.26" width="0" layer="19" extent="1-1"/>
+<contactref element="R12" pad="1"/>
+<wire x1="-41.59" y1="-162.56" x2="-42.91" y2="-175.26" width="0" layer="19" extent="1-1"/>
+<wire x1="-30.48" y1="-115.57" x2="-41.59" y2="-162.56" width="0" layer="19" extent="1-1"/>
 <wire x1="-30.48" y1="-107.95" x2="-30.48" y2="-115.57" width="0" layer="19" extent="1-1"/>
 <wire x1="-14.09" y1="14.47" x2="-30.48" y2="-107.95" width="0" layer="19" extent="1-1"/>
@@
 <signal name="SW_R">
 <contactref element="X1" pad="7"/>
+<contactref element="R16" pad="2"/>
+<wire x1="-29.09" y1="6.47" x2="-61.28" y2="-248.92" width="0" layer="19" extent="1-1"/>
 </signal>
 <signal name="N$12">
@@
 <wire x1="-39.37" y1="-195.145" x2="-41.59" y2="-199.39" width="0" layer="19" extent="1-1"/>
 </signal>
+<signal name="N$13">
+<contactref element="OK1" pad="6"/>
+<contactref element="R15" pad="2"/>
+<wire x1="-73.98" y1="-205.74" x2="-39.37" y2="-185.855" width="0" layer="19" extent="1-1"/>
+</signal>
+<signal name="A2_LIVE_IN">
+<contactref element="R15" pad="1"/>
+<contactref element="T1" pad="A1"/>
+<contactref element="R17" pad="1"/>
+<contactref element="T2" pad="A1"/>
+<wire x1="-66.548" y1="-234.95" x2="-56.83" y2="-248.92" width="0" layer="19" extent="1-1"/>
+<wire x1="-75.88" y1="-205.74" x2="-66.548" y2="-234.95" width="0" layer="19" extent="1-1"/>
+<wire x1="-66.548" y1="-191.77" x2="-75.88" y2="-205.74" width="0" layer="19" extent="1-1"/>
+</signal>
+<signal name="N$14">
+<contactref element="T1" pad="G"/>
+<contactref element="OK1" pad="4"/>
+<wire x1="-34.29" y1="-185.855" x2="-55.372" y2="-191.77" width="0" layer="19" extent="1-1"/>
+</signal>
+<signal name="A1_LIVE_OUT">
+<contactref element="T1" pad="A2"/>
+<contactref element="T2" pad="A2"/>
+<wire x1="-60.96" y1="-234.95" x2="-60.96" y2="-191.77" width="0" layer="19" extent="1-1"/>
+</signal>
+<signal name="N$15">
+<contactref element="R16" pad="1"/>
+<contactref element="OK2" pad="1"/>
+<wire x1="-63.18" y1="-248.92" x2="-72.39" y2="-256.105" width="0" layer="19" extent="1-1"/>
+</signal>
+<signal name="N$16">
+<contactref element="OK2" pad="6"/>
+<contactref element="R17" pad="2"/>
+<wire x1="-54.93" y1="-248.92" x2="-72.39" y2="-246.815" width="0" layer="19" extent="1-1"/>
+</signal>
+<signal name="N$17">
+<contactref element="T2" pad="G"/>
+<contactref element="OK2" pad="4"/>
+<wire x1="-55.372" y1="-234.95" x2="-67.31" y2="-246.815" width="0" layer="19" extent="1-1"/>
+</signal>
+<signal name="LIVE_IN">
+<contactref element="C8" pad="1"/>
+</signal>
 </signals>
